Commit message: feat(sim): adapt SO101 MuJoCo inference and add control panel
- so101.xml.template: jaw euler MuJoCo-only calibration (+0.209440 rad);
  timestep=0.001, noslip_iterations=20, cone=elliptic for stable grasping
- so101_base.xacro / so101_ros2_control.xacro: MujocoSystemInterface plugin
  wiring; mujoco_model_path injected via xacro at launch
- mujoco_adapter: YAML-driven camera injection, Gazebo→MuJoCo RPY
  conversion, camera_publish_rate derived from peripherals fps (no SSOT)
- camera_presets.py: MuJoCo-native preset values; description.py: pass
  mujoco_model_path into URDF xacro
- model_infer_panel.py: Klein-blue web panel (port 8766); START/STOP
  inference, random banana placement, reset scene, AutoTest; SSE log
  stream
- action_dispatcher: inference_timeout_sec watchdog (default 10s);
  idempotent start/stop; stall diagnostic log; f-string fixes
- action_dispatch README: updated service docs and architecture notes
- robot_config README: replace dual_camera_monitor section with
  model_infer_panel + Rerun visualization guidance

Co-Authored-By: Claude Sonnet 4.6

Co-Authored-By: GPT-5.5

File: src/robot_description/urdf/lerobot/so101/so101_base.xacro (robot description, xacro)
@@ -341,5 +341,5 @@
 	<!-- Joint from gripper to jaw -->
 	<joint name="6" type="revolute">
-		<origin xyz="0.0202 0.0188 -0.0234" rpy="1.5708 -5.14108e-17 -1.38655e-14" />
+		<origin xyz="0.0202 0.0188 -0.0234" rpy="1.5708 0.209440 0.000001" />
 		<parent link="gripper" />
 		<child link="jaw" />

File: src/robot_description/urdf/lerobot/so101/so101_ros2_control.xacro (robot description, xacro)
@@ -9,4 +9,5 @@
     <xacro:arg name="sim_plugin" default="gz_ros2_control/GazeboSimSystem"/>
     <xacro:arg name="mujoco_model" default=""/>
+    <xacro:arg name="camera_publish_rate" default=""/>
     <ros2_control name="RobotSystem" type="system">
         <xacro:if value="$(arg use_sim)">
@@ -15,4 +16,7 @@
                 <xacro:if value="${'$(arg mujoco_model)' != ''}">
                     <param name="mujoco_model">$(arg mujoco_model)</param>
+                </xacro:if>
+                <xacro:if value="${'$(arg camera_publish_rate)' != ''}">
+                    <param name="camera_publish_rate">$(arg camera_publish_rate)</param>
                 </xacro:if>
             </hardware>
